File: KiCad/USB PD/USB PD.kicad_sch (KiCad schematic)
At the start: 37 parts, among them J10 CFG, J11 SEL, J12 GND, J7 VCC, J8 ESP32 Jumpers, J8 TX, J9 RX, U1 AO3400A, U2 IP2721, U4 TYPE-C_6P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

Commit message: Added reverse polarity protection
Parts:
- removed TP3: TestPoint, Library:TestPoint_THTPad_2.0x2.0mm_Drill1.0mm, symbol Connector:TestPoint
Connections:
- net 5V OUT: now also TP5.1
- net at R1.1, R1.2, U5.4 (VSENSE): no longer TP5.1
Changed lines of the file:
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@@
   (junction (at 153.67 120.015) (diameter 0) (color 0 0 0 0)
   )
+  (junction (at 223.52 112.395) (diameter 0) (color 0 0 0 0)
+  )
   (junction (at 132.08 53.34) (diameter 0) (color 0 0 0 0)
   )
@@
   )
   (junction (at 217.17 112.395) (diameter 0) (color 0 0 0 0)
-  )
-  (junction (at 203.2 127.635) (diameter 0) (color 0 0 0 0)
   )
   (junction (at 135.89 53.34) (diameter 0) (color 0 0 0 0)
@@
     (stroke (width 0) (type default))
   )
-  (wire (pts (xy 217.17 112.395) (xy 240.03 112.395))
-    (stroke (width 0) (type default))
-  )
   (wire (pts (xy 138.43 127.635) (xy 138.43 131.445))
     (stroke (width 0) (type default))
@@
     (stroke (width 0) (type default))
   )
+  (wire (pts (xy 223.52 112.395) (xy 240.03 112.395))
+    (stroke (width 0) (type default))
+  )
   (wire (pts (xy 158.75 71.12) (xy 169.545 71.12))
     (stroke (width 0) (type default))
@@
     (stroke (width 0) (type default))
   )
-  (wire (pts (xy 203.2 127.635) (xy 191.77 127.635))
+  (wire (pts (xy 191.77 127.635) (xy 217.17 127.635))
     (stroke (width 0) (type default))
   )
@@
     (stroke (width 0) (type default))
   )
+  (wire (pts (xy 223.52 112.395) (xy 217.17 112.395))
+    (stroke (width 0) (type default))
+  )
   (wire (pts (xy 245.11 36.83) (xy 245.11 49.53))
     (stroke (width 0) (type default))
@@
   )
   (wire (pts (xy 156.21 102.235) (xy 199.39 102.235))
-    (stroke (width 0) (type default))
-  )
-  (wire (pts (xy 217.17 127.635) (xy 203.2 127.635))
     (stroke (width 0) (type default))
   )
@@
         (path "/339a92df-fdbb-48aa-b235-136f297cfd8f"
           (reference "J8") (unit 1)
-        )
-      )
-    )
-  )
-  (symbol (lib_id "Connector:TestPoint") (at 196.85 27.94 0) (mirror y) (unit 1)
-    (in_bom no) (on_board yes) (dnp no) (fields_autoplaced)
-    (property "Reference" "TP3" (at 195.453 23.9943 0)
-      (effects (font (size 1.27 1.27)) (justify left))
-    )
-    (property "Value" "TestPoint" (at 195.453 25.9153 0)
-      (effects (font (size 1.27 1.27)) (justify left))
-    )
-    (property "Footprint" "Library:TestPoint_THTPad_2.0x2.0mm_Drill1.0mm" (at 191.77 27.94 0)
-      (effects (font (size 1.27 1.27)) hide)
-    )
-    (property "Datasheet" "~" (at 191.77 27.94 0)
-      (effects (font (size 1.27 1.27)) hide)
-    )
-    (pin "1")
-    (instances
-      (project "USB PD"
-        (path "/339a92df-fdbb-48aa-b235-136f297cfd8f"
-          (reference "TP3") (unit 1)
         )
       )
@@
         (path "/339a92df-fdbb-48aa-b235-136f297cfd8f"
           (reference "H4") (unit 1)
+        )
+      )
+    )
+  )
+  (symbol (lib_id "Connector:TestPoint") (at 223.52 112.395 0) (mirror y) (unit 1)
+    (in_bom no) (on_board yes) (dnp no)
+    (property "Reference" "TP5" (at 222.123 108.4493 0)
+      (effects (font (size 1.27 1.27)) (justify left))
+    )
+    (property "Value" "TestPoint" (at 222.123 110.3703 0)
+      (effects (font (size 1.27 1.27)) (justify left))
+    )
+    (property "Footprint" "Library:TestPoint_THTPad_2.0x2.0mm_Drill1.0mm" (at 218.44 112.395 0)
+      (effects (font (size 1.27 1.27)) hide)
+    )
+    (property "Datasheet" "~" (at 218.44 112.395 0)
+      (effects (font (size 1.27 1.27)) hide)
+    )
+    (pin "1")
+    (instances
+      (project "Retro Display Module"
+        (path "/046eef48-6d3f-4288-a12a-fc20b7e12e30"
+          (reference "TP5") (unit 1)
+        )
+      )
+      (project "USB PD"
+        (path "/339a92df-fdbb-48aa-b235-136f297cfd8f"
+          (reference "TP3") (unit 1)
         )
       )
@@
         )
       )
-    )
-  )
-  (symbol (lib_id "Connector:TestPoint") (at 203.2 127.635 0) (mirror x) (unit 1)
-    (in_bom no) (on_board yes) (dnp no)
-    (property "Reference" "TP5" (at 204.597 131.5807 0)
-      (effects (font (size 1.27 1.27)) (justify left))
-    )
-    (property "Value" "TestPoint" (at 204.597 129.6597 0)
-      (effects (font (size 1.27 1.27)) (justify left))
-    )
-    (property "Footprint" "Library:TestPoint_THTPad_2.0x2.0mm_Drill1.0mm" (at 208.28 127.635 0)
-      (effects (font (size 1.27 1.27)) hide)
-    )
-    (property "Datasheet" "~" (at 208.28 127.635 0)
-      (effects (font (size 1.27 1.27)) hide)
-    )
-    (pin "1")
-    (instances
-      (project "Retro Display Module"
-        (path "/046eef48-6d3f-4288-a12a-fc20b7e12e30"
-          (reference "TP5") (unit 1)
-        )
-      )
-      (project "USB PD"
-        (path "/339a92df-fdbb-48aa-b235-136f297cfd8f"
-          (reference "TP4") (unit 1)
-        )
-      )
